File: power.kicad_sch (KiCad schematic)
At the start: 13 parts, among them J1 +12V, 2.1mm, Q1 DMP3013SFV, U2 AP1509-50

Commit message: power stuff. 2.5, 1.2 for switch
Parts:
- removed TP1: TestPoint, KiCad/kicad-footprints/TestPoint.pretty:TestPoint_Pad_D1.5mm, symbol Connector:TestPoint
- removed TP2: TestPoint, KiCad/kicad-footprints/TestPoint.pretty:TestPoint_Pad_D1.0mm, symbol Connector:TestPoint
- added C10, C7: 100pF, symbol Device:C
- added C11, C6, C8, C9: 22uF, symbol Device:C
- added C5: 330uF, KiCad/kicad-footprints/Capacitor_Tantalum_SMD.pretty:CP_EIA-7343-43_Kemet-X_Pad2.25x2.55mm_HandSolder, symbol Device:CP
- added D3: SS34, KiCad/Diodes_SMD.pretty:D_SMA_Handsoldering, symbol Device:D_Schottky
- added F1: 2016L260/24MR, symbol Device:Polyfuse
- added J2: +5V, KiCad/Pin_Headers.pretty:Pin_Header_Straight_1x03_Pitch2.54mm, symbol Connector_Generic:Conn_01x03
- added J3: +3.3V, KiCad/Pin_Headers.pretty:Pin_Header_Straight_1x03_Pitch2.54mm, symbol Connector_Generic:Conn_01x03
- added J3: +12V, KiCad/Pin_Headers.pretty:Pin_Header_Straight_1x03_Pitch2.54mm, symbol Connector_Generic:Conn_01x03
- added L2: 47uH, KiCad/kicad-footprints/Inductor_SMD.pretty:L_10.4x10.4_H4.8, symbol Device:L
- added L2: 1.2uH, KiCad/kicad-footprints/Inductor_SMD.pretty:L_10.4x10.4_H4.8, symbol Device:L
- added L3: 2.2uH, KiCad/kicad-footprints/Inductor_SMD.pretty:L_10.4x10.4_H4.8, symbol Device:L
- added R2, R3, R5: 150k, symbol Device:R
- added R4: 475k, symbol Device:R
- added U2: AP1509-33, KiCad/kicad-footprints/Package_SO.pretty:SOIC-8_3.9x4.9mm_P1.27mm, symbol CustomSymbols:AP1509
- added U3, U4: PAM2310, KiCad/kicad-footprints/Package_SO.pretty:Diodes_SO-8EP, symbol CustomSymbols:PAM2310
- L1: value 47uH -> 2.2uH
- renumbered C5 to C4, U2 to U1
Connections:
- net +12V: now also J3.1 (Pin_1), J3.2 (Pin_2), J3.3 (Pin_3), U2.1 (VIN)
- net +5V: now also C6.1, C9.1, J2.1 (Pin_1), J2.2 (Pin_2), J2.3 (Pin_3), U3.2 (VIN), U3.7 (EN), U4.2 (VIN), U4.7 (EN)
- net GND: now also C2.2, D1.2 (A), Q1.4 (G), R1.1, C11.1, C5.2, C6.2, C8.1, C9.2, D3.2 (A), R3.2, R5.2, U2.4 (SD), U2.5 (GND), U2.6 (GND), U2.7 (GND), U2.8 (GND), U3.4 (GND), U4.4 (GND)
- net at C1.1, Q1.5 (D): now also F1.2; no longer J1.1
- new net: F1.1, J1.1
- new net: D3.1 (K), L2.1, U2.2 (Output)
- new net: R2.2, R3.1
- new net: R4.2, R5.1
- new net: U3.1 (NC), U3.6 (NC), U3.8 (NC)
- new net: L2.1, U3.3 (SW)
- new net: C7.1, U3.5 (FB)
- new net: U4.1 (NC), U4.6 (NC), U4.8 (NC)
- new net: L3.1, U4.3 (SW)
- new net: C10.1, U4.5 (FB)
- new net +1.2V: C7.2, C8.2, L2.2, R2.1
- new net +2.5V: C10.2, C11.2, L3.2, R4.1
- new net +3.3V: C5.1, J3.1 (Pin_1), J3.2 (Pin_2), J3.3 (Pin_3), L2.2, U2.3 (FB)
Other:
- note added: "1.2V"
- note added: "2.5V"
- note added: "3.3V"
- note added: "3.3V 2A"
- note added: "5V"
- moved on the sheet: C1, C2, C3, C4, D1, D2, J1, L1, Q1, R1
